File: BadgeSam.sch (KiCad schematic (older format))
At the start: 6 parts

Commit message: add r g b and button
Parts:
- added C?: C, symbol Device:C
- added SW?: SW_Push, symbol Switch:SW_Push
Connections:
- net labels added: +3.3V, B2, B3, B4, G2, G3, G4, R2, R3, R4, RST
- wire segments 22 -> 41
Changed lines of the file:
@@
 EESchema Schematic File Version 4
+LIBS:power
+LIBS:device
+LIBS:74xx
+LIBS:audio
+LIBS:interface
 EELAYER 30 0
 EELAYER END
@@
 	8680 2770 8680 2675
 Text Label 7855 2570 0    50   ~ 0
-R1
+R2
 Text Label 7860 2770 0    50   ~ 0
-G1
+G2
 Text Label 7870 2970 0    50   ~ 0
-B1
+B3
 $Comp
 L Device:LED_RGBA D?
@@
 	8680 3735 8680 3640
 Text Label 7855 3535 0    50   ~ 0
-R1
+R3
 Text Label 7860 3735 0    50   ~ 0
-G1
+G3
 Text Label 7870 3935 0    50   ~ 0
-B1
+B3
 $Comp
 L Device:LED_RGBA D?
@@
 	8675 4705 8675 4610
 Text Label 7850 4505 0    50   ~ 0
-R1
+R4
 Text Label 7855 4705 0    50   ~ 0
-G1
+G4
 Text Label 7865 4905 0    50   ~ 0
-B1
+B4
 Wire Wire Line
 	1430 2895 1430 2805
@@
 $EndComp
 $Comp
+L MCU_ST_STM8:STM8S003F3P U?
+U 1 1 5E3DBFB6
+P 3570 3170
+F 0 "U?" H 3320 4110 50  0000 C CNN
+F 1 "STM8S003F3P" H 3885 4105 50  0000 C CNN
+F 2 "Package_SO:TSSOP-20_4.4x6.5mm_P0.65mm" H 3620 4270 50  0001 L CNN
+F 3 "http://www.st.com/st-web-ui/static/active/en/resource/technical/document/datasheet/DM00024550.pdf" H 3520 2770 50  0001 C CNN
+	1    3570 3170
+	1    0    0    -1
+$EndComp
+$Comp
+L Device:C C?
+U 1 1 5E45D8AC
+P 4875 3075
+F 0 "C?" H 4990 3121 50  0000 L CNN
+F 1 "C" H 4990 3030 50  0000 L CNN
+F 2 "" H 4913 2925 50  0001 C CNN
+F 3 "~" H 4875 3075 50  0001 C CNN
+	1    4875 3075
+	1    0    0    -1
+$EndComp
+$Comp
 L power:GND #PWR?
 U 1 1 5E3DA5A2
@@
 $EndComp
 $Comp
-L MCU_ST_STM8:STM8S003F3P U?
-U 1 1 5E3DBFB6
-P 3570 3170
-F 0 "U?" H 3320 4110 50  0000 C CNN
-F 1 "STM8S003F3P" H 3885 4105 50  0000 C CNN
-F 2 "Package_SO:TSSOP-20_4.4x6.5mm_P0.65mm" H 3620 4270 50  0001 L CNN
-F 3 "http://www.st.com/st-web-ui/static/active/en/resource/technical/document/datasheet/DM00024550.pdf" H 3520 2770 50  0001 C CNN
-	1    3570 3170
-	1    0    0    -1
-$EndComp
+L power:GND #PWR?
+U 1 1 5E45DFCD
+P 4875 3375
+F 0 "#PWR?" H 4875 3125 50  0001 C CNN
+F 1 "GND" H 4880 3202 50  0000 C CNN
+F 2 "" H 4875 3375 50  0001 C CNN
+F 3 "" H 4875 3375 50  0001 C CNN
+	1    4875 3375
+	1    0    0    -1
+$EndComp
+$Comp
+L power:+3.3V #PWR?
+U 1 1 5E45E9D8
+P 4875 2800
+F 0 "#PWR?" H 4875 2650 50  0001 C CNN
+F 1 "+3.3V" H 4890 2973 50  0000 C CNN
+F 2 "" H 4875 2800 50  0001 C CNN
+F 3 "" H 4875 2800 50  0001 C CNN
+	1    4875 2800
+	1    0    0    -1
+$EndComp
+Wire Wire Line
+	4875 2925 4875 2800
+Wire Wire Line
+	4875 3375 4875 3225
+$Comp
+L power:GND #PWR?
+U 1 1 5E45FD96
+P 3570 4250
+F 0 "#PWR?" H 3570 4000 50  0001 C CNN
+F 1 "GND" H 3575 4077 50  0000 C CNN
+F 2 "" H 3570 4250 50  0001 C CNN
+F 3 "" H 3570 4250 50  0001 C CNN
+	1    3570 4250
+	1    0    0    -1
+$EndComp
+Wire Wire Line
+	3570 4250 3570 4170
+$Comp
+L power:+3.3V #PWR?
+U 1 1 5E462D8E
+P 3570 2050
+F 0 "#PWR?" H 3570 1900 50  0001 C CNN
+F 1 "+3.3V" H 3585 2223 50  0000 C CNN
+F 2 "" H 3570 2050 50  0001 C CNN
+F 3 "" H 3570 2050 50  0001 C CNN
+	1    3570 2050
+	1    0    0    -1
+$EndComp
+Wire Wire Line
+	3570 2050 3570 2170
+Text Label 2910 2470 0    50   ~ 0
+R1
+Wire Wire Line
+	2910 2470 2970 2470
+Text Label 2910 2570 0    50   ~ 0
+G1
+Wire Wire Line
+	2910 2570 2970 2570
+Text Label 2900 2670 0    50   ~ 0
+B1
+Wire Wire Line
+	2900 2670 2970 2670
+Text Label 2880 2870 0    50   ~ 0
+R2
+Wire Wire Line
+	2880 2870 2970 2870
+Text Label 2890 2970 0    50   ~ 0
+G2
+Wire Wire Line
+	2970 2970 2890 2970
+Text Label 2880 3170 0    50   ~ 0
+B2
+Wire Wire Line
+	2970 3170 2880 3170
+Text Label 2880 3270 0    50   ~ 0
+R3
+Text Label 2880 3370 0    50   ~ 0
+G3
+Text Label 2880 3470 0    50   ~ 0
+B3
+Text Label 2880 3570 0    50   ~ 0
+R4
+Text Label 4230 2870 0    50   ~ 0
+G4
+Text Label 4240 2970 0    50   ~ 0
+B4
+Wire Wire Line
+	2880 3270 2970 3270
+Wire Wire Line
+	2970 3370 2880 3370
+Wire Wire Line
+	2880 3470 2970 3470
+Wire Wire Line
+	2970 3570 2880 3570
+Wire Wire Line
+	4240 2970 4170 2970
+Wire Wire Line
+	4230 2870 4170 2870
+Text Label 2890 3770 0    50   ~ 0
+RST
+$Comp
+L Switch:SW_Push SW?
+U 1 1 5E477841
+P 2590 3770
+F 0 "SW?" H 2590 4055 50  0000 C CNN
+F 1 "SW_Push" H 2590 3964 50  0000 C CNN
+F 2 "" H 2590 3970 50  0001 C CNN
+F 3 "~" H 2590 3970 50  0001 C CNN
+	1    2590 3770
+	1    0    0    -1
+$EndComp
+Wire Wire Line
+	2790 3770 2970 3770
+Wire Wire Line
+	2390 3770 2310 3770
+Wire Wire Line
+	2310 3770 2310 3950
+$Comp
+L power:GND #PWR?
+U 1 1 5E47A567
+P 2310 3950
+F 0 "#PWR?" H 2310 3700 50  0001 C CNN
+F 1 "GND" H 2315 3777 50  0000 C CNN
+F 2 "" H 2310 3950 50  0001 C CNN
+F 3 "" H 2310 3950 50  0001 C CNN
+	1    2310 3950
+	1    0    0    -1
+$EndComp

Commit message: battery
Parts:
- added C?: 1uF, symbol Device:C_Small
- added R?: 10K, symbol Device:R_Small
- C?: value C -> 0.1uF
- SW?: value SW_Push -> RESET
Connections:
- net labels removed: +3.3V
- wire segments 41 -> 48
Other:
- moved on the sheet: SW?
Changed lines of the file:
@@
 EESchema Schematic File Version 4
-LIBS:power
-LIBS:device
-LIBS:74xx
-LIBS:audio
-LIBS:interface
 EELAYER 30 0
 EELAYER END
@@
 P 4875 3075
 F 0 "C?" H 4990 3121 50  0000 L CNN
-F 1 "C" H 4990 3030 50  0000 L CNN
+F 1 "0.1uF" H 4990 3030 50  0000 L CNN
 F 2 "" H 4913 2925 50  0001 C CNN
 F 3 "~" H 4875 3075 50  0001 C CNN
@@
 	1    0    0    -1
 $EndComp
-$Comp
-L power:+3.3V #PWR?
-U 1 1 5E45E9D8
-P 4875 2800
-F 0 "#PWR?" H 4875 2650 50  0001 C CNN
-F 1 "+3.3V" H 4890 2973 50  0000 C CNN
-F 2 "" H 4875 2800 50  0001 C CNN
-F 3 "" H 4875 2800 50  0001 C CNN
-	1    4875 2800
-	1    0    0    -1
-$EndComp
 Wire Wire Line
 	4875 2925 4875 2800
@@
 Wire Wire Line
 	3570 4250 3570 4170
-$Comp
-L power:+3.3V #PWR?
-U 1 1 5E462D8E
-P 3570 2050
-F 0 "#PWR?" H 3570 1900 50  0001 C CNN
-F 1 "+3.3V" H 3585 2223 50  0000 C CNN
-F 2 "" H 3570 2050 50  0001 C CNN
-F 3 "" H 3570 2050 50  0001 C CNN
-	1    3570 2050
-	1    0    0    -1
-$EndComp
 Wire Wire Line
 	3570 2050 3570 2170
@@
 Wire Wire Line
 	4230 2870 4170 2870
-Text Label 2890 3770 0    50   ~ 0
-RST
 $Comp
 L Switch:SW_Push SW?
 U 1 1 5E477841
-P 2590 3770
-F 0 "SW?" H 2590 4055 50  0000 C CNN
-F 1 "SW_Push" H 2590 3964 50  0000 C CNN
-F 2 "" H 2590 3970 50  0001 C CNN
-F 3 "~" H 2590 3970 50  0001 C CNN
-	1    2590 3770
-	1    0    0    -1
-$EndComp
-Wire Wire Line
-	2790 3770 2970 3770
-Wire Wire Line
-	2390 3770 2310 3770
-Wire Wire Line
-	2310 3770 2310 3950
+P 1435 4155
+F 0 "SW?" H 1435 4440 50  0000 C CNN
+F 1 "RESET" H 1435 4349 50  0000 C CNN
+F 2 "" H 1435 4355 50  0001 C CNN
+F 3 "~" H 1435 4355 50  0001 C CNN
+	1    1435 4155
+	1    0    0    -1
+$EndComp
+Wire Wire Line
+	1635 4155 1660 4155
+Wire Wire Line
+	1235 4155 1155 4155
+Wire Wire Line
+	1155 4155 1155 4335
 $Comp
 L power:GND #PWR?
 U 1 1 5E47A567
-P 2310 3950
-F 0 "#PWR?" H 2310 3700 50  0001 C CNN
-F 1 "GND" H 2315 3777 50  0000 C CNN
-F 2 "" H 2310 3950 50  0001 C CNN
-F 3 "" H 2310 3950 50  0001 C CNN
-	1    2310 3950
-	1    0    0    -1
-$EndComp
+P 1155 4335
+F 0 "#PWR?" H 1155 4085 50  0001 C CNN
+F 1 "GND" H 1160 4162 50  0000 C CNN
+F 2 "" H 1155 4335 50  0001 C CNN
+F 3 "" H 1155 4335 50  0001 C CNN
+	1    1155 4335
+	1    0    0    -1
+$EndComp
+$Comp
+L Device:C_Small C?
+U 1 1 5E45F30C
+P 2915 4020
+F 0 "C?" H 3007 4066 50  0000 L CNN
+F 1 "1uF" H 3007 3975 50  0000 L CNN
+F 2 "" H 2915 4020 50  0001 C CNN
+F 3 "~" H 2915 4020 50  0001 C CNN
+	1    2915 4020
+	1    0    0    -1
+$EndComp
+Wire Wire Line
+	2970 3870 2915 3870
+Wire Wire Line
+	2915 3870 2915 3920
+Wire Wire Line
+	2915 4120 2915 4200
+$Comp
+L power:GND #PWR?
+U 1 1 5E461CF3
+P 2915 4200
+F 0 "#PWR?" H 2915 3950 50  0001 C CNN
+F 1 "GND" H 2920 4027 50  0000 C CNN
+F 2 "" H 2915 4200 50  0001 C CNN
+F 3 "" H 2915 4200 50  0001 C CNN
+	1    2915 4200
+	1    0    0    -1
+$EndComp
+$Comp
+L Device:R_Small R?
+U 1 1 5E46267A
+P 1660 4020
+F 0 "R?" H 1719 4066 50  0000 L CNN
+F 1 "10K" H 1719 3975 50  0000 L CNN
+F 2 "" H 1660 4020 50  0001 C CNN
+F 3 "~" H 1660 4020 50  0001 C CNN
+	1    1660 4020
+	1    0    0    -1
+$EndComp
+Wire Wire Line
+	1660 4120 1660 4155
+Connection ~ 1660 4155
+Wire Wire Line
+	1660 4155 1815 4155
+Wire Wire Line
+	1660 3920 1660 3875
+Wire Wire Line
+	2970 3770 2900 3770
+Text Label 2900 3770 0    50   ~ 0
+RST
+Text Label 1815 4155 0    50   ~ 0
+RST
+$Comp
+L power:+BATT #PWR?
+U 1 1 5E46D9B9
+P 1660 3875
+F 0 "#PWR?" H 1660 3725 50  0001 C CNN
+F 1 "+BATT" H 1675 4048 50  0000 C CNN
+F 2 "" H 1660 3875 50  0001 C CNN
+F 3 "" H 1660 3875 50  0001 C CNN
+	1    1660 3875
+	1    0    0    -1
+$EndComp
+$Comp
+L power:+BATT #PWR?
+U 1 1 5E46F2BE
+P 4875 2800
+F 0 "#PWR?" H 4875 2650 50  0001 C CNN
+F 1 "+BATT" H 4890 2973 50  0000 C CNN
+F 2 "" H 4875 2800 50  0001 C CNN
+F 3 "" H 4875 2800 50  0001 C CNN
+	1    4875 2800
+	1    0    0    -1
+$EndComp
+$Comp
+L power:+BATT #PWR?
+U 1 1 5E46F805
+P 3570 2050
+F 0 "#PWR?" H 3570 1900 50  0001 C CNN
+F 1 "+BATT" H 3585 2223 50  0000 C CNN
+F 2 "" H 3570 2050 50  0001 C CNN
+F 3 "" H 3570 2050 50  0001 C CNN
+	1    3570 2050
+	1    0    0    -1
+$EndComp
+$Comp
+L power:+BATT #PWR?
+U 1 1 5E47165E
+P 8665 1630
+F 0 "#PWR?" H 8665 1480 50  0001 C CNN
+F 1 "+BATT" H 8680 1803 50  0000 C CNN
+F 2 "" H 8665 1630 50  0001 C CNN
+F 3 "" H 8665 1630 50  0001 C CNN
+	1    8665 1630
+	1    0    0    -1
+$EndComp
+$Comp
+L power:+BATT #PWR?
+U 1 1 5E471FC1
+P 8680 2675
+F 0 "#PWR?" H 8680 2525 50  0001 C CNN
+F 1 "+BATT" H 8695 2848 50  0000 C CNN
+F 2 "" H 8680 2675 50  0001 C CNN
+F 3 "" H 8680 2675 50  0001 C CNN
+	1    8680 2675
+	1    0    0    -1
+$EndComp
+$Comp
+L power:+BATT #PWR?
+U 1 1 5E472AC9
+P 8680 3640
+F 0 "#PWR?" H 8680 3490 50  0001 C CNN
+F 1 "+BATT" H 8695 3813 50  0000 C CNN
+F 2 "" H 8680 3640 50  0001 C CNN
+F 3 "" H 8680 3640 50  0001 C CNN
+	1    8680 3640
+	1    0    0    -1
+$EndComp

Commit message: add library for badge sam and battery holder
Parts:
- BT1: renamed from BT?; footprint (none) -> BadgeSam:79523141
- C1, C2: renamed from C?; footprint (none) -> Capacitor_SMD:C_0805_2012Metric_Pad1.15x1.40mm_HandSolder
- D1, D2, D3, D4: renamed from D?; manf# (none) -> 155124M173200A
- R1: renamed from R?; footprint (none) -> Resistor_SMD:R_0805_2012Metric_Pad1.15x1.40mm_HandSolder
- SW1: renamed from SW?; footprint (none) -> Button_Switch_SMD:SW_SPST_TL3342
- gave numbers to parts that had none: 1
Connections:
- net labels added: PC6, PC7, SWIM
- wire segments 48 -> 51
Other:
- note added: "PD1 has SWIM interface"
- moved on the sheet: BT1, C1, C2, R1, SW1, U1

Commit message: define size
Parts:
- D1, D2, D3, D4: footprint (none) -> BadgeSam:LED_155124M173200
Changed lines of the file:
@@
 EESchema Schematic File Version 4
+LIBS:BadgeSam-cache
 EELAYER 30 0
 EELAYER END
@@
 F 0 "D1" H 8190 2222 50  0000 C CNN
 F 1 "LED_RGBA" H 8190 2131 50  0000 C CNN
-F 2 "" H 8190 1675 50  0001 C CNN
+F 2 "BadgeSam:LED_155124M173200" H 8190 1675 50  0001 C CNN
 F 3 "~" H 8190 1675 50  0001 C CNN
 F 4 "155124M173200A" H 8190 1725 50  0001 C CNN "manf#"
@@
 F 0 "D3" H 8205 3267 50  0000 C CNN
 F 1 "LED_RGBA" H 8205 3176 50  0000 C CNN
-F 2 "" H 8205 2720 50  0001 C CNN
+F 2 "BadgeSam:LED_155124M173200" H 8205 2720 50  0001 C CNN
 F 3 "~" H 8205 2720 50  0001 C CNN
 F 4 "155124M173200A" H 8205 2770 50  0001 C CNN "manf#"
@@
 F 0 "D4" H 8205 4232 50  0000 C CNN
 F 1 "LED_RGBA" H 8205 4141 50  0000 C CNN
-F 2 "" H 8205 3685 50  0001 C CNN
+F 2 "BadgeSam:LED_155124M173200" H 8205 3685 50  0001 C CNN
 F 3 "~" H 8205 3685 50  0001 C CNN
 F 4 "155124M173200A" H 8205 3735 50  0001 C CNN "manf#"
@@
 F 0 "D2" H 8200 5202 50  0000 C CNN
 F 1 "LED_RGBA" H 8200 5111 50  0000 C CNN
-F 2 "" H 8200 4655 50  0001 C CNN
+F 2 "BadgeSam:LED_155124M173200" H 8200 4655 50  0001 C CNN
 F 3 "~" H 8200 4655 50  0001 C CNN
 F 4 "155124M173200A" H 8200 4705 50  0001 C CNN "manf#"

Commit message: change rgb and footprint led
Parts:
- removed D1, D2, D3, D4: LED_RGBA, BadgeSam:LED_155124M173200, symbol Device:LED_RGBA
- added D1, D2, D3, D4: LED_ARGB, BadgeSam:156120M173000, symbol Device:LED_ARGB
Connections:
- wire segments 51 -> 50
- no-connect marks 0 -> 1
Changed lines of the file:
@@
 $EndDescr
-$Comp
-L Device:LED_RGBA D1
-U 1 1 5E3CB5F4
-P 8190 1725
-F 0 "D1" H 8190 2222 50  0000 C CNN
-F 1 "LED_RGBA" H 8190 2131 50  0000 C CNN
-F 2 "BadgeSam:LED_155124M173200" H 8190 1675 50  0001 C CNN
-F 3 "~" H 8190 1675 50  0001 C CNN
-F 4 "155124M173200A" H 8190 1725 50  0001 C CNN "manf#"
-	1    8190 1725
-	1    0    0    -1
-$EndComp
 $Comp
 L Device:Battery_Cell BT1
@@
 Text Label 7855 1925 0    50   ~ 0
 B1
-$Comp
-L Device:LED_RGBA D3
-U 1 1 5E3D361F
-P 8205 2770
-F 0 "D3" H 8205 3267 50  0000 C CNN
-F 1 "LED_RGBA" H 8205 3176 50  0000 C CNN
-F 2 "BadgeSam:LED_155124M173200" H 8205 2720 50  0001 C CNN
-F 3 "~" H 8205 2720 50  0001 C CNN
-F 4 "155124M173200A" H 8205 2770 50  0001 C CNN "manf#"
-	1    8205 2770
-	1    0    0    -1
-$EndComp
 Wire Wire Line
 	8005 2570 7855 2570
@@
 Text Label 7870 2970 0    50   ~ 0
 B3
-$Comp
-L Device:LED_RGBA D4
-U 1 1 5E3D490E
-P 8205 3735
-F 0 "D4" H 8205 4232 50  0000 C CNN
-F 1 "LED_RGBA" H 8205 4141 50  0000 C CNN
-F 2 "BadgeSam:LED_155124M173200" H 8205 3685 50  0001 C CNN
-F 3 "~" H 8205 3685 50  0001 C CNN
-F 4 "155124M173200A" H 8205 3735 50  0001 C CNN "manf#"
-	1    8205 3735
-	1    0    0    -1
-$EndComp
 Wire Wire Line
 	8005 3535 7855 3535
@@
 Text Label 7870 3935 0    50   ~ 0
 B3
-$Comp
-L Device:LED_RGBA D2
-U 1 1 5E3D63B2
-P 8200 4705
-F 0 "D2" H 8200 5202 50  0000 C CNN
-F 1 "LED_RGBA" H 8200 5111 50  0000 C CNN
-F 2 "BadgeSam:LED_155124M173200" H 8200 4655 50  0001 C CNN
-F 3 "~" H 8200 4655 50  0001 C CNN
-F 4 "155124M173200A" H 8200 4705 50  0001 C CNN "manf#"
-	1    8200 4705
-	1    0    0    -1
-$EndComp
 Wire Wire Line
 	8000 4505 7850 4505
@@
 $EndComp
 $Comp
-L MCU_ST_STM8:STM8S003F3P U1
-U 1 1 5E3DBFB6
-P 5000 2195
-F 0 "U1" H 4750 3135 50  0000 C CNN
-F 1 "STM8S003F3P" H 5315 3130 50  0000 C CNN
-F 2 "Package_SO:TSSOP-20_4.4x6.5mm_P0.65mm" H 5050 3295 50  0001 L CNN
-F 3 "http://www.st.com/st-web-ui/static/active/en/resource/technical/document/datasheet/DM00024550.pdf" H 4950 1795 50  0001 C CNN
-	1    5000 2195
-	1    0    0    -1
-$EndComp
-$Comp
 L Device:C C2
 U 1 1 5E45D8AC
@@
 Text Label 4330 1695 2    50   ~ 0
 R1
-Wire Wire Line
-	4340 1495 4400 1495
 Text Label 4340 1495 2    50   ~ 0
 G1
-Wire Wire Line
-	4340 1595 4400 1595
 Text Label 4340 1595 2    50   ~ 0
 B1
-Wire Wire Line
-	4330 1695 4400 1695
 Text Label 4310 2395 2    50   ~ 0
 R2
 Text Label 4330 1895 2    50   ~ 0
 G2
-Wire Wire Line
-	4400 2195 4310 2195
-Text Label 4045 2290 2    50   ~ 0
+Text Label 4310 2295 2    50   ~ 0
 G3
 Text Label 5670 1995 0    50   ~ 0
@@
 B4
 Wire Wire Line
-	4310 2295 4400 2295
-Wire Wire Line
-	4400 2395 4310 2395
-Wire Wire Line
-	4310 2495 4400 2495
-Wire Wire Line
-	4400 2595 4310 2595
-Wire Wire Line
 	5670 1995 5600 1995
 $Comp
@@
 $EndComp
 Wire Wire Line
-	4400 2895 4345 2895
-Wire Wire Line
 	4345 2895 4345 2945
 Wire Wire Line
@@
 Wire Wire Line
 	3360 1115 3360 1070
-Wire Wire Line
-	4400 2795 4330 2795
 Text Label 4330 2795 2    50   ~ 0
 RST
@@
 Wire Wire Line
 	5600 1895 5670 1895
-Wire Wire Line
-	4400 1895 4330 1895
-Wire Wire Line
-	4330 1995 4400 1995
-Text Label 3840 2525 2    50   ~ 0
+Text Label 4310 2495 2    50   ~ 0
 PC6
-Text Label 3775 2735 2    50   ~ 0
+Text Label 4310 2595 2    50   ~ 0
 PC7
 Wire Wire Line
@@
 Text Label 5670 1895 0    50   ~ 0
 SWIM
+$Comp
+L Device:LED_ARGB D3
+U 1 1 5E4E5EE2
+P 8205 2770
+F 0 "D3" H 8205 3267 50  0000 C CNN
+F 1 "LED_ARGB" H 8205 3176 50  0000 C CNN
+F 2 "BadgeSam:156120M173000" H 8205 2720 50  0001 C CNN
+F 3 "~" H 8205 2720 50  0001 C CNN
+	1    8205 2770
+	1    0    0    -1
+$EndComp
+$Comp
+L Device:LED_ARGB D4
+U 1 1 5E4DD52A
+P 8205 3735
+F 0 "D4" H 8205 4232 50  0000 C CNN
+F 1 "LED_ARGB" H 8205 4141 50  0000 C CNN
+F 2 "BadgeSam:156120M173000" H 8205 3685 50  0001 C CNN
+F 3 "~" H 8205 3685 50  0001 C CNN
+	1    8205 3735
+	1    0    0    -1
+$EndComp
+$Comp
+L Device:LED_ARGB D2
+U 1 1 5E4DE527
+P 8200 4705
+F 0 "D2" H 8200 5202 50  0000 C CNN
+F 1 "LED_ARGB" H 8200 5111 50  0000 C CNN
+F 2 "BadgeSam:156120M173000" H 8200 4655 50  0001 C CNN
+F 3 "~" H 8200 4655 50  0001 C CNN
+	1    8200 4705
+	1    0    0    -1
+$EndComp
+$Comp
+L Device:LED_ARGB D1
+U 1 1 5E4DF060
+P 8190 1725
+F 0 "D1" H 8190 2222 50  0000 C CNN
+F 1 "LED_ARGB" H 8190 2131 50  0000 C CNN
+F 2 "BadgeSam:156120M173000" H 8190 1675 50  0001 C CNN
+F 3 "~" H 8190 1675 50  0001 C CNN
+	1    8190 1725
+	1    0    0    -1
+$EndComp
+$Comp
+L power:+BATT #PWR01
+U 1 1 5E4EFB6E
+P 8675 4610
+F 0 "#PWR01" H 8675 4460 50  0001 C CNN
+F 1 "+BATT" H 8690 4783 50  0000 C CNN
+F 2 "" H 8675 4610 50  0001 C CNN
+F 3 "" H 8675 4610 50  0001 C CNN
+	1    8675 4610
+	1    0    0    -1
+$EndComp
+NoConn ~ 4400 2195
+Wire Wire Line
+	4400 2595 4310 2595
+Wire Wire Line
+	4310 2495 4400 2495
+Wire Wire Line
+	4400 2395 4310 2395
+Wire Wire Line
+	4310 2295 4400 2295
+Wire Wire Line
+	4400 1895 4330 1895
+Wire Wire Line
+	4330 1995 4400 1995
+Wire Wire Line
+	4330 1695 4400 1695
+Wire Wire Line
+	4400 2895 4345 2895
+Wire Wire Line
+	4340 1595 4400 1595
+Wire Wire Line
+	4340 1495 4400 1495
+Wire Wire Line
+	4400 2795 4330 2795
+$Comp
+L MCU_ST_STM8:STM8S003F3P U1
+U 1 1 5E3DBFB6
+P 5000 2195
+F 0 "U1" H 4750 3135 50  0000 C CNN
+F 1 "STM8S003F3P" H 5315 3130 50  0000 C CNN
+F 2 "Package_SO:TSSOP-20_4.4x6.5mm_P0.65mm" H 5050 3295 50  0001 L CNN
+F 3 "http://www.st.com/st-web-ui/static/active/en/resource/technical/document/datasheet/DM00024550.pdf" H 4950 1795 50  0001 C CNN
+	1    5000 2195
+	1    0    0    -1
+$EndComp
 $EndSCHEMATC

Commit message: routeo and pin prog
Parts:
- added J1: PROG, Connector_PinHeader_2.54mm:PinHeader_1x04_P2.54mm_Vertical, symbol Connector:Conn_01x04_Female
Connections:
- net +BATT: now also J1.4 (Pin_4)
- net B2: now also D3.4 (BK)
- net B3: no longer D3.4 (BK)
- net GND: now also J1.2 (Pin_2)
- net RST: now also J1.1 (Pin_1)
- net SWIM: now also J1.3 (Pin_3)
- net PC6: no longer names the net of U1.16 (PC6)
- net PC7: no longer names the net of U1.17 (PC7)
- no-connect marks 1 -> 3
Changed lines of the file:
@@
 G2
 Text Label 7870 2970 0    50   ~ 0
-B3
+B2
 Wire Wire Line
 	8005 3535 7855 3535
@@
 Wire Wire Line
 	5600 1895 5670 1895
-Text Label 4310 2495 2    50   ~ 0
-PC6
-Text Label 4310 2595 2    50   ~ 0
-PC7
 Wire Wire Line
 	3360 1840 3360 2035
@@
 NoConn ~ 4400 2195
 Wire Wire Line
-	4400 2595 4310 2595
-Wire Wire Line
-	4310 2495 4400 2495
-Wire Wire Line
 	4400 2395 4310 2395
 Wire Wire Line
@@
 	1    0    0    -1
 $EndComp
+$Comp
+L Connector:Conn_01x04_Female J1
+U 1 1 5E50F491
+P 3255 3530
+F 0 "J1" H 3283 3506 50  0000 L CNN
+F 1 "PROG" H 3283 3415 50  0000 L CNN
+F 2 "Connector_PinHeader_2.54mm:PinHeader_1x04_P2.54mm_Vertical" H 3255 3530 50  0001 C CNN
+F 3 "~" H 3255 3530 50  0001 C CNN
+	1    3255 3530
+	1    0    0    -1
+$EndComp
+Text Label 2925 3430 0    50   ~ 0
+RST
+Text Label 2900 3630 0    50   ~ 0
+SWIM
+$Comp
+L power:+BATT #PWR02
+U 1 1 5E511BE3
+P 2675 3705
+F 0 "#PWR02" H 2675 3555 50  0001 C CNN
+F 1 "+BATT" H 2690 3878 50  0000 C CNN
+F 2 "" H 2675 3705 50  0001 C CNN
+F 3 "" H 2675 3705 50  0001 C CNN
+	1    2675 3705
+	1    0    0    -1
+$EndComp
+Wire Wire Line
+	3055 3630 2900 3630
+Wire Wire Line
+	3055 3430 2925 3430
+$Comp
+L power:GND #PWR03
+U 1 1 5E5173CA
+P 2845 3820
+F 0 "#PWR03" H 2845 3570 50  0001 C CNN
+F 1 "GND" H 2850 3647 50  0000 C CNN
+F 2 "" H 2845 3820 50  0001 C CNN
+F 3 "" H 2845 3820 50  0001 C CNN
+	1    2845 3820
+	1    0    0    -1
+$EndComp
+Wire Wire Line
+	2845 3820 2845 3530
+Wire Wire Line
+	2845 3530 3055 3530
+Wire Wire Line
+	2675 3730 2675 3705
+Wire Wire Line
+	2675 3730 3055 3730
+NoConn ~ 4400 2495
+NoConn ~ 4400 2595
 $EndSCHEMATC

Commit message: Fix leds and traces
Connections:
- net B1: now also U1.3 (PD6); no longer U1.6 (PA2)
- net B2: now also U1.15 (PC5); no longer U1.11 (PB5)
- net B3: now also U1.17 (PC7); no longer U1.19 (PD2)
- net B4: now also U1.1 (PD4); no longer U1.2 (PD5)
- net G1: now also U1.6 (PA2); no longer U1.5 (PA1)
- net G2: now also U1.14 (PC4); no longer U1.12 (PB4)
- net G3: now also U1.19 (PD2); no longer U1.14 (PC4)
- net G4: now also U1.2 (PD5); no longer U1.1 (PD4)
- net R1: now also U1.5 (PA1); no longer U1.10 (PA3)
- net R2: now also U1.13 (PC3); no longer U1.15 (PC5)
- net R4: now also U1.16 (PC6); no longer U1.3 (PD6)
Changed lines of the file:
@@
 EESchema Schematic File Version 4
-LIBS:BadgeSam-cache
 EELAYER 30 0
 EELAYER END
@@
 Wire Wire Line
 	5000 1075 5000 1195
-Text Label 4330 1695 2    50   ~ 0
+Text Label 4340 1495 2    50   ~ 0
 R1
-Text Label 4340 1495 2    50   ~ 0
-G1
-Text Label 4340 1595 2    50   ~ 0
-B1
-Text Label 4310 2395 2    50   ~ 0
+Text Label 4310 2195 2    50   ~ 0
 R2
-Text Label 4330 1895 2    50   ~ 0
+Text Label 4310 2295 2    50   ~ 0
 G2
-Text Label 4310 2295 2    50   ~ 0
+Text Label 5670 1995 0    50   ~ 0
 G3
-Text Label 5670 1995 0    50   ~ 0
+Text Label 4310 2595 2    50   ~ 0
 B3
-Text Label 5670 2395 0    50   ~ 0
+Text Label 4310 2495 2    50   ~ 0
 R4
+Text Label 5670 2295 0    50   ~ 0
+G4
 Text Label 5670 2195 0    50   ~ 0
-G4
-Text Label 5670 2295 0    50   ~ 0
 B4
 Wire Wire Line
@@
 Wire Wire Line
 	5670 2095 5600 2095
-Text Label 4330 1995 2    50   ~ 0
+Text Label 4310 2395 2    50   ~ 0
 B2
 Text Label 5670 2095 0    50   ~ 0
@@
 	1    0    0    -1
 $EndComp
-NoConn ~ 4400 2195
 Wire Wire Line
 	4400 2395 4310 2395
 Wire Wire Line
 	4310 2295 4400 2295
-Wire Wire Line
-	4400 1895 4330 1895
-Wire Wire Line
-	4330 1995 4400 1995
-Wire Wire Line
-	4330 1695 4400 1695
 Wire Wire Line
 	4400 2895 4345 2895
@@
 Wire Wire Line
 	2675 3730 3055 3730
-NoConn ~ 4400 2495
-NoConn ~ 4400 2595
+Wire Wire Line
+	4310 2595 4400 2595
+Text Label 5670 2395 0    50   ~ 0
+B1
+Text Label 4340 1595 2    50   ~ 0
+G1
+Wire Wire Line
+	4400 2495 4310 2495
+Wire Wire Line
+	4400 2195 4310 2195
+NoConn ~ 4400 1895
+NoConn ~ 4400 1995
+NoConn ~ 4400 1695
 $EndSCHEMATC
